File: Hardware/Schematic.sch (EAGLE design)
At the start: 103 parts, among them IC1 XC6220A331MR-G, IC2 BD5229G-TR, J1 FH34SRJ-24S-0.5SH_99_, J2 SAMACSYS_PARTS_USB4110-GF-ACP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, J3 QWIIC_RIGHT_ANGLE, J4 112A-TAAR-R03_ATTEND, Q1 20V/4.2A/52mΩ/1.4W, Q2 20V/4.2A/52mΩ/1.4W, Q3 SI1308EDL-T1-GE3, U1 MAX17048G+T10, U2 ESP32-C6-WROOM-1-N8, U3 DS3231SN#, U4 W25Q512JVEIQ

Commit message: updated sschematic and board
Parts:
- C1_BAT: value (none) -> 4.7uF
- C3: value (none) -> 100uF
- renumbered TP1 to TX, TP10 to EPD_CS, TP12 to EPD_RST, TP13 to EPD_3V3_C, TP14 to V_BUS, TP15 to INT_RTC, TP16 to 3V3, TP17 to EPD_3V3, TP2 to RX, TP3 to V_BAT, TP4 to GND_1, TP5 to GND_2, TP6 to MISO, TP7 to MOSI, TP8 to SCK, TP9 to EPD_BUSY
Other:
- note added: "BATTERY CHARGE LEVEL"
- note added: "DISPLAY TYPE SELECTOR"
- note added: "E-PAPER DISPLAY HEADER"
- note added: "ENVIRONMENTAL SENSOR"
- note added: "EPAPER DRIVE CIRCUIT"
- note added: "EPD POWER"
- note added: "ESP32 C6"
- note added: "EXTERNAL NOR FLASH 64MB"
- note added: "LDO VOLTAGE REGULATOR"
- note added: "LI-PO BATTERY CHARGING CONTROLLER"
- note added: "RTC MODULE"
- note added: "SD CARD"
- note added: "SPI ESD PROTECTION LINES"
- note added: "TEST PADS"
- note added: "USB-C CONNECTOR & ESD PROTECTION"
- note added: "VOLTAGE SUPERVISOR + RESET & BOOT / IO BUTTON"
